Commit message: Have the tf from frames local to the autorally working

File: autorally/autorally_description/urdf/autoRallyPlatform_with_sensors2.urdf.xacro (robot description, xacro)
@@ -22,4 +22,6 @@
 -->
 <robot name="autorally_platform" xmlns:xacro="http://www.ros.org/wiki/xacro">
+  <!-- sensor Configuration -->
+  <xacro:property name="use_cameras" value="false"/>
   <!-- Degree-to-radian conversions -->
   <xacro:property name="degrees_45" value="0.785398163"/>
@@ -366,4 +368,5 @@
     <child link="imu_link"/>
   </joint>
+<xacro:if value="${use_cameras}">
   <joint name="camera_joint" type="fixed">
     <axis xyz="0 0 -1" />
@@ -520,4 +523,5 @@
     </sensor>
   </gazebo>
+</xacro:if>
   <!-- Wheels -->
   <xacro:front_wheel lr_prefix="left" fr_prefix="front"
@@ -556,5 +560,68 @@
     </sensor>
   </gazebo>
+  <!-- Hokuo Laser Joint -->
+  <joint name="hokuyo_joint" type="fixed">
+    <axis xyz="0 0 -1" />
+    <origin xyz=".14 0 .2" rpy="0 0 0"/>
+    <parent link="base_link"/>
+    <child link ="hokuyo"/>
+  </joint>
+  <!-- Hokuyo Laser -->
+  <link name="hokuyo">
+    <collision>
+      <origin xyz="0 0 0" rpy="0 0 0"/>
+      <geometry>
+    <box size="0.1 0.1 0.1"/>
+      </geometry>
+    </collision>
+    <visual>
+      <origin xyz="0 0 0" rpy="0 0 0"/>
+      <geometry>
+        <mesh filename="package://autorally_description/urdf/hokuyo.dae"/>
+      </geometry>
+    </visual>
+    <inertial>
+      <mass value="1e-5" />
+      <origin xyz="0 0 0" rpy="0 0 0"/>
+      <inertia ixx="1e-6" ixy="0" ixz="0" iyy="1e-6" iyz="0" izz="1e-6" />
+    </inertial>
+  </link>
+  <gazebo reference="hokuyo">
+    <sensor type="ray" name="laser">
+      <pose>0 0 0 0 0 0</pose>
+      <visualize>true</visualize>
+      <update_rate>40</update_rate>
+      <ray>
+        <scan>
+          <horizontal>
+            <samples>720</samples>
+            <resolution>1</resolution>
+            <min_angle>-1.570796</min_angle>
+            <max_angle>1.570796</max_angle>
+          </horizontal>
+        </scan>
+        <range>
+          <min>0.10</min>
+          <max>30.0</max>
+          <resolution>0.01</resolution>
+        </range>
+        <noise>
+          <type>gaussian</type>
+          <!-- Noise parameters based on published spec for Hokuyo laser
+               achieving "+-30mm" accuracy at range < 10m.  A mean of 0.0m and
+               stddev of 0.01m will put 99.7% of samples within 0.03m of the true
+               reading. -->
+          <mean>0.0</mean>
+          <stddev>0.01</stddev>
+        </noise>
+      </ray>
+      <plugin name="hokuyo_node" filename="libgazebo_ros_laser.so">
+        <topicName>/lidar_front</topicName>
+         <frameName>hokuyo</frameName>
+      </plugin>
+    </sensor>
+</gazebo>
   <!-- Forward facing Lidar Sensor -->
+<!--
   <xacro:include filename="$(find ardupilot_sitl_gazebo_plugin)/urdf/sensors/lidar_sensor.urdf.xacro" />
   <xacro:lidar_sensor
@@ -572,4 +639,5 @@
     <origin xyz="0.5 0 0.1" rpy="0 0 0"/>
   </xacro:lidar_sensor>
+-->
   <gazebo>
     <plugin name="gazebo_ros_control" filename="libgazebo_ros_control.so">

File: autorally/autorally_description/urdf/autoRallyTrack_scaled.urdf (robot description, URDF)
Before this commit: robot track, 1 links, 0 joints
Links:
- link track_link: geometry collision mesh filename=package://autorally_description/urdf/autoRallyTrack.stl scale=0.03 0.03 0.10; visual mesh filename=package://autorally_description/urdf/autoRallyTrack.stl scale=0.03 0.03 0.10

Commit message: Most of the ROS navigation stack is now working with the Autorally platform. Including nodes: map_server, amcl, and move base (which provides both the local and global cost maps). Move base might need some tweeks when it comes to path planning yet. The base controller node (for translating twist msgs to chassisCommand msgs) is not implemented yet.

File: autorally/autorally_description/urdf/autoRallyPlatform_with_sensors2.urdf.xacro (robot description, xacro)
@@ -549,6 +549,6 @@
     <alwaysOn>true</alwaysOn>
     <updateRate>50.0</updateRate>
-    <bodyName>chassis</bodyName>
-    <topicName>odom</topicName>
+    <bodyName>base_link</bodyName>
+    <topicName>ground_truth/state</topicName>
     <gaussianNoise>0.01</gaussianNoise>
     <frameName>world</frameName>
@@ -573,5 +573,5 @@
   <joint name="hokuyo_joint" type="fixed">
     <axis xyz="0 0 -1" />
-    <origin xyz=".14 0 .2" rpy="0 0 0"/>
+    <origin xyz=".17 0 .2" rpy="0 0 0"/>
     <parent link="base_link"/>
     <child link ="hokuyo"/>
