Commit message: initial commit on branch - replaced autorally-indigo repo with autorally-kinetic repo

File: autorally/autorally_description/urdf/autoRallyPlatform.urdf.xacro (robot description, xacro)
@@ -91,4 +91,6 @@
   <xacro:property name="servo_stall_torque" value="3.432620346181713"/>
   <xacro:property name="servo_no_load_speed" value="8.05536578"/>
+  <!-- arg to specify namespace -->
+  <xacro:arg name="prefix" default=""/>
   <material name="chassis_mat">
     <color rgba="0.5 0.5 0.5 1"/>
@@ -139,10 +141,10 @@
       <type>transmission_interface/SimpleTransmission</type>
       <joint name="${lr_prefix}_${fr_prefix}_shock">
-        <hardwareInterface>EffortJointInterface</hardwareInterface>
+        <hardwareInterface>hardware_interface/EffortJointInterface</hardwareInterface>
       </joint>
       <actuator name="${lr_prefix}_${fr_prefix}_shock_act">
         <!-- This hardwareInterface element exists for compatibility
              with ROS Hydro. -->
-        <hardwareInterface>EffortJointInterface</hardwareInterface>
+        <hardwareInterface>hardware_interface/EffortJointInterface</hardwareInterface>
         <mechanicalReduction>1</mechanicalReduction>
       </actuator>
@@ -166,10 +168,10 @@
       <type>transmission_interface/SimpleTransmission</type>
       <joint name="${lr_prefix}_${fr_prefix}_shock">
-        <hardwareInterface>EffortJointInterface</hardwareInterface>
+        <hardwareInterface>hardware_interface/EffortJointInterface</hardwareInterface>
       </joint>
       <actuator name="${lr_prefix}_${fr_prefix}_shock_act">
         <!-- This hardwareInterface element exists for compatibility
              with ROS Hydro. -->
-        <hardwareInterface>EffortJointInterface</hardwareInterface>
+        <hardwareInterface>hardware_interface/EffortJointInterface</hardwareInterface>
         <mechanicalReduction>1</mechanicalReduction>
       </actuator>
@@ -199,10 +201,10 @@
       <type>transmission_interface/SimpleTransmission</type>
       <joint name="${lr_prefix}_${fr_prefix}_axle">
-        <hardwareInterface>EffortJointInterface</hardwareInterface>
+        <hardwareInterface>hardware_interface/EffortJointInterface</hardwareInterface>
       </joint>
       <actuator name="${lr_prefix}_${fr_prefix}_axle_act">
         <!-- This hardwareInterface element exists for compatibility
              with ROS Hydro. -->
-        <hardwareInterface>EffortJointInterface</hardwareInterface>
+        <hardwareInterface>hardware_interface/EffortJointInterface</hardwareInterface>
         <mechanicalReduction>1</mechanicalReduction>
       </actuator>
@@ -270,10 +272,10 @@
       <type>transmission_interface/SimpleTransmission</type>
       <joint name="${lr_prefix}_steering_joint">
-        <hardwareInterface>EffortJointInterface</hardwareInterface>
+        <hardwareInterface>hardware_interface/EffortJointInterface</hardwareInterface>
       </joint>
       <actuator name="${lr_prefix}_steering_act">
         <!-- This hardwareInterface element exists for compatibility
              with ROS Hydro. -->
-        <hardwareInterface>EffortJointInterface</hardwareInterface>
+        <hardwareInterface>hardware_interface/EffortJointInterface</hardwareInterface>
         <mechanicalReduction>1</mechanicalReduction>
       </actuator>
@@ -347,4 +349,21 @@
     <child link="chassis"/>
   </joint>
+  <link name="gps_link">
+    <collision>
+      <geometry>
+        <box size="0.1 0.1 0.1"/>
+      </geometry>
+    </collision>
+    <inertial>
+      <mass value="1e-5" />
+      <origin xyz="0 0 0" rpy="0 0 0"/>
+      <inertia ixx="1e-6" ixy="0" ixz="0" iyy="1e-6" iyz="0" izz="1e-6" />
+    </inertial>
+  </link>
+  <joint name="gps_joint" type="fixed">
+    <origin xyz="-0.36 0 0.1359" rpy="0 0 0"/>
+    <parent link="base_link"/>
+    <child link="gps_link"/>
+  </joint>
   <link name="imu_link">
     <collision>
@@ -361,5 +380,5 @@
   </link>
   <joint name="imu_joint" type="fixed">
-    <origin xyz="0 0 0" rpy="0 0 0"/>
+    <origin xyz="-0.039 0 0.0859" rpy="0 0 0"/>
     <parent link="base_link"/>
     <child link="imu_link"/>
@@ -367,7 +386,45 @@
   <joint name="camera_joint" type="fixed">
     <axis xyz="0 0 -1" />
-    <origin xyz="0.12 0 0.05" rpy="0 0 0"/>
+    <origin xyz="0.127 0 0.2159" rpy="0 0 0"/>
     <parent link="base_link"/>
     <child link="camera_link"/>
+  </joint>
+ <!-- <link name="odom">
+    <collision>
+      <origin xyz="0 0 0" rpy="0 0 0"/>
+      <geometry>
+        <box size="0.1 0.1 0.1"/>
+      </geometry>
+    </collision>
+    <inertial>
+      <mass value="1e-5" />
+      <origin xyz="0 0 0" rpy="0 0 0"/>
+      <inertia ixx="1e-6" ixy="0" ixz="0" iyy="1e-6" iyz="0" izz="1e-6" />
+    </inertial>
+  </link>
+  <joint name="odom_joint" type="fixed">
+    <axis xyz="0 0 0" />
+    <origin xyz="0 0 0" rpy="0 0 0"/>
+    <parent link="odom"/>
+    <child link="base_link"/>
+  </joint>
+-->
+ <link name="odom_ground_truth">
+    <collision>
+      <geometry>
+        <box size="0.1 0.1 0.1"/>
+      </geometry>
+    </collision>
+    <inertial>
+      <mass value="1e-5" />
+      <origin xyz="0 0 0" rpy="0 0 0"/>
+      <inertia ixx="1e-6" ixy="0" ixz="0" iyy="1e-6" iyz="0" izz="1e-6" />
+    </inertial>
+  </link>
+  <joint name="odom_ground_truth_joint" type="fixed">
+    <axis xyz="0 0 0" />
+    <origin xyz="-0.039 0 0.0859" rpy="0 0 0"/>
+    <parent link="base_link"/>
+    <child link="odom_ground_truth"/>
   </joint>
   <!-- Camera -->
@@ -379,6 +436,5 @@
       </geometry>
     </collision>
-<!--
-    <visual>
+    <!--<visual>
       <origin xyz="0 0 0" rpy="0 0 0"/>
       <geometry>
@@ -386,34 +442,5 @@
       </geometry>
       <material name="red"/>
-    </visual>
--->
-    <inertial>
-      <mass value="1e-5" />
-      <origin xyz="0 0 0" rpy="0 0 0"/>
-      <inertia ixx="1e-6" ixy="0" ixz="0" iyy="1e-6" iyz="0" izz="1e-6" />
-    </inertial>
-  </link>
-  <joint name="side_camera_joint" type="fixed">
-    <axis xyz="0 1 0" />
-    <origin xyz="0 -3 0" rpy="0 0 1.5708"/>
-    <parent link="base_link"/>
-    <child link="side_camera_link"/>
-  </joint>
-  <!-- Camera -->
-  <link name="side_camera_link">
-    <!-- <collision>
-      <origin xyz="0 0 0" rpy="0 0 0"/>
-      <geometry>
-        <box size="0.05 0.05 0.05"/>
-      </geometry>
-    </collision>
-    <visual>
-      <origin xyz="0 0 0" rpy="0 0 0"/>
-      <geometry>
-        <box size="0.05 0.05 0.05"/>
-      </geometry>
-      <material name="red"/>
-    </visual>
-    -->
+    </visual>-->
     <inertial>
       <mass value="1e-5" />
@@ -446,5 +473,5 @@
       <camera name="right">
         <pose>0.02 -0.07 0 0 0 0</pose>
-        <horizontal_fov>3.0</horizontal_fov>
+        <horizontal_fov>1.3962634</horizontal_fov>
         <image>
           <width>1280</width>
@@ -463,4 +490,5 @@
       </camera>
       <plugin name="stereo_camera_controller" filename="libgazebo_ros_multicamera.so">
+        <robotNamespace>$(arg prefix)</robotNamespace>
         <alwaysOn>true</alwaysOn>
         <updateRate>60.0</updateRate>
@@ -475,44 +503,4 @@
         <distortionK3>-0.000165</distortionK3>
         <distortionT1>-0.000336</distortionT1>
-        <distortionT2>0.0</distortionT2> -->
-      </plugin>
-    </sensor>
-  </gazebo>
-   <!-- camera -->
-  <gazebo reference="side_camera_link">
-    <sensor type="camera" name="camera_side">
-      <update_rate>30.0</update_rate>
-      <camera name="side">
-        <horizontal_fov>1.3962634</horizontal_fov>
-        <image>
-          <width>1280</width>
-          <height>1024</height>
-          <format>R8G8B8</format>
-        </image>
-        <clip>
-          <near>0.02</near>
-          <far>50</far>
-        </clip>
-        <noise>
-          <type>gaussian</type>
-          <!-- Noise is sampled independently per pixel on each frame.
-               That pixel's noise value is added to each of its color
-               channels, which at that point lie in the range [0,1]. -->
-          <mean>0.0</mean>
-          <stddev>0.007</stddev>
-        </noise>
-      </camera>
-      <plugin name="camera_controller" filename="libgazebo_ros_camera.so">
-        <alwaysOn>true</alwaysOn>
-        <updateRate>0.0</updateRate>
-        <cameraName>camera_side</cameraName>
-        <imageTopicName>image_raw</imageTopicName>
-        <cameraInfoTopicName>camera_info</cameraInfoTopicName>
-        <frameName>side_camera_link</frameName>
-        <hackBaseline>0.07</hackBaseline>
-        <!-- <distortionK1>0.0</distortionK1>
-        <distortionK2>0.0</distortionK2>
-        <distortionK3>0.0</distortionK3>
-        <distortionT1>0.0</distortionT1>
         <distortionT2>0.0</distortionT2> -->
       </plugin>
@@ -542,14 +530,14 @@
   <gazebo>
     <plugin name="gazebo_ros_control" filename="libgazebo_ros_control.so">
-      <robotNamespace>/autorally_platform</robotNamespace>
+      <robotNamespace>$(arg prefix)</robotNamespace>
       <robotSimType>gazebo_ros_control/DefaultRobotHWSim</robotSimType>
     </plugin>
     <plugin name="imu" filename="libhector_gazebo_ros_imu.so">
-      <robotNamespace>/autorally_platform</robotNamespace>
-      <serviceName>/imu/calibrate</serviceName>
+      <robotNamespace>$(arg prefix)</robotNamespace>
+      <serviceName>$(arg prefix)/imu/calibrate</serviceName>
       <updateRate>200.0</updateRate>
       <bodyName>imu_link</bodyName>
       <frameId>imu_link</frameId>
-      <topicName>imu</topicName>
+      <topicName>imu/imu</topicName>
       <rpyOffset>0 0 0</rpyOffset>
       <xyzOffset>0 0 0</xyzOffset>
@@ -566,7 +554,8 @@
     </plugin>
     <plugin name="gps" filename="libhector_gazebo_ros_gps.so">
+      <robotNamespace>$(arg prefix)</robotNamespace>
       <updateRate>20.0</updateRate>
-      <bodyName>base_link</bodyName>
-      <frameId>base_link</frameId>
+      <bodyName>gps_link</bodyName>
+      <frameId>gps_link</frameId>
       <topicName>gpsRoverStatus</topicName>
       <velocityTopicName>fix_velocity</velocityTopicName>
@@ -579,5 +568,16 @@
       <velocityGaussianNoise>0.005 0.005 0.05</velocityGaussianNoise>
     </plugin>
-    <!-- <plugin name="tire_friction" filename="libTireFrictionPlugin.so">
+    <plugin name="p3d_base_controller" filename="libgazebo_ros_p3d.so">
+      <alwaysOn>true</alwaysOn>
+      <updateRate>200.0</updateRate>
+      <bodyName>odom_ground_truth</bodyName>
+      <topicName>ground_truth/state_raw</topicName>
+      <gaussianNoise>0.00</gaussianNoise>
+      <frameName>world</frameName>
+      <!-- origin is at spawn location -->
+      <xyzOffset>0 8.5 0</xyzOffset>
+      <rpyOffset>0 0 0</rpyOffset>
+    </plugin>
+    <!--<plugin name="tire_friction" filename="libTireFrictionPlugin.so">
       <link_name>left_rear_wheel</link_name>
       <collision_name>collision</collision_name>
@@ -587,5 +587,5 @@
       <slip_dynamic>0.20</slip_dynamic>
       <speed_static>0.50</speed_static>
-    </plugin> -->
+    </plugin>-->
   </gazebo>
 </robot>
