Commit message: Moved files from tmp-storage, moved base_controller... to msu_autorally_helper

File: msu_autorally/msu_autorally_helper/models/autoRallyTrack.urdf (robot description, URDF)
Before this commit: robot track, 1 links, 0 joints
Links:
- link track_link: geometry collision mesh filename=package://autorally_description/urdf/autoRallyTrack.stl scale=0.01 0.01 0.01; visual mesh filename=package://autorally_description/urdf/autoRallyTrack.stl scale=0.01 0.01 0.01
